Commit message: [urdf] generate urdf

File: models/iRonCub-Mk1_1_v1/iRonCub/robots/iRonCub-Mk1_1_Gazebo_v1/model_stl.urdf (robot description, URDF)
Before this commit: robot iCub, 97 links, 96 joints
Joints:
- joint imu_frame_fixed_joint: origin xyz=0.009500000190735 0.13344313685842288 0.00929998892871537 rpy=3.141592653589793 1.570796289791727 -1.5707963237945508 -> xyz=0.009500000190735 0.13344313685842288 0.00929998892871537 rpy=3.141592653589793 1.5707962897917267 -1.5707963267948966
- joint l_arm_ft_sensor: origin xyz=0.05093014324520241 0 0.029175829465898032 rpy=0 -1.3089969894682865 3.1415926535896164 -> xyz=0.05093014324520241 0 0.029175829465898032 rpy=0 -1.3089969894682862 3.1415926535896137
- joint l_elbow: origin xyz=0 -0.02000000036832994 0.0792599999070578 rpy=0 -1.3089969894682885 -3.1415926535896865 -> xyz=0 -0.020000000368329995 0.07925999990705779 rpy=0 -1.308996989468288 -3.1415926535896834
- joint l_hip_roll: origin xyz=0 0.044099999999999986 0 rpy=0 0 0 -> xyz=0 0.04409999999999999 0 rpy=0 0 0
- joint l_leg_ft_sensor: origin xyz=-0.0008301999999999962 7.519999999999749e-05 -0.07429999999999995 rpy=3.141592653589793 0 0 -> xyz=-0.0008301999999999962 7.519999999998361e-05 -0.07429999999999995 rpy=3.141592653589793 0 0
- joint l_shoulder_roll: axis -0.2588190174889569 -1.1253323287226445e-17 0.9659259953138497 -> -0.2588190174889569 -1.0645723802156837e-17 0.9659259953138496
- joint l_shoulder_yaw: axis 0.9659258393523219 -5.74303850210394e-15 0.2588189963497913 -> 0.9659258393523219 -5.743038501910067e-15 0.2588189963497913; origin xyz=0.025313329844247154 1.2922216940935982e-07 -0.005396821114290115 rpy=-0.2526895449300091 -0.00851861944331826 -0.06703989350788468 -> xyz=0.025313329844247154 1.2922216939548203e-07 -0.005396821114290115 rpy=-0.2526895449300091 -0.00851861944331826 -0.06703989350788468
- joint neck_roll: axis 0.0 1.8017533007091882e-10 0.9999999628183933 -> 0.0 1.8017532951719595e-10 0.9999999628183934
- joint neck_yaw: axis 0.0 0.9999999628183934 -1.8017532951839303e-10 -> 0.0 0.9999999628183934 -1.8017532951719595e-10
- joint r_elbow_turbine: origin xyz=-0.25731143930868927 0.07362600000000007 0.09741646806310904 rpy=1.291296957309416 -0.3534717274196087 -1.4717699551817651 -> xyz=-0.25731143930868927 0.07362600000000005 0.09741646806310904 rpy=1.291296957309416 -0.3534717274196087 -1.4717699551817651
- joint r_jet_turbine: origin xyz=-0.169999999809265 -0.1141002 -0.1158885 rpy=-1.5707963207923916 -0.9424794397774846 -3.1415926514080383 -> xyz=-0.169999999809265 -0.1141002 -0.1158885 rpy=-1.5707963207923927 -0.9424794397774842 -3.141592651408038
- joint r_lower_leg_skin_14_fixed_joint: origin xyz=0.05504769999999998 -0.031175900000000006 -0.02190000000000003 rpy=-3.141591818848249 -1.4650273563521197 -0.6540334071673023 -> xyz=0.05504769999999998 -0.031175900000000006 -0.02190000000000003 rpy=-3.1415918188482506 -1.46502735635212 -0.6540334071673009
- joint r_lower_leg_skin_17_fixed_joint: origin xyz=0.027874999999999976 -0.05031190000000001 -0.023882000000000014 rpy=-3.141564526201752 -1.563662402374811 -1.1802250875588731 -> xyz=0.027874999999999976 -0.05031190000000001 -0.023882000000000014 rpy=-3.1415645262018144 -1.5636624023748111 -1.180225087558763
- joint r_lower_leg_skin_19_fixed_joint: origin xyz=0.03575341 0.041062799999999997 0.006064999999999987 rpy=-8.908777174257102e-07 -1.4349869697782824 -2.1586361801672447 -> xyz=0.03575341 0.041062799999999997 0.006064999999999987 rpy=-8.908777145556939e-07 -1.434986969778283 -2.158636180167247
- joint r_lower_leg_skin_20_fixed_joint: origin xyz=0.0234419 0.047990799999999986 -0.004952000000000012 rpy=-3.2055654966350685e-06 -1.5001551303072314 -1.8675509241250097 -> xyz=0.0234419 0.047990799999999986 -0.004952000000000012 rpy=-3.2055655052862463e-06 -1.500155130307231 -1.867550924125001
- joint r_lower_leg_skin_21_fixed_joint: origin xyz=0.024270400000000004 0.04853779999999998 -0.024276999999999993 rpy=2.2967114955750172e-05 -1.5554551388057172 -1.8741197231626954 -> xyz=0.024270400000000004 0.04853779999999998 -0.024276999999999993 rpy=2.2967114934038522e-05 -1.5554551388057167 -1.8741197231626947
- joint r_lower_leg_skin_31_fixed_joint: origin xyz=0.03914639999999998 -0.042270899999999986 0.006327000000000027 rpy=-6.583817471389409e-07 -1.4186494462021593 2.2085303298592955 -> xyz=0.03914639999999998 -0.042270899999999986 0.006327000000000027 rpy=-6.583817537316898e-07 -1.4186494462021593 2.2085303298593018
- joint r_lower_leg_skin_32_fixed_joint: origin xyz=0.045983029999999994 0.03258469999999997 -0.080733 rpy=-3.141590149878832 -1.5223828979770995 0.6459403808870791 -> xyz=0.045983029999999994 0.03258469999999997 -0.080733 rpy=-3.1415901498788155 -1.5223828979770997 0.6459403808870626
- joint r_lower_leg_skin_36_fixed_joint: origin xyz=0.05322409999999998 -0.015601800000000027 -0.088362 rpy=-3.141590341443774 -1.5158726528065043 -0.20740733566009956 -> xyz=0.05322409999999998 -0.015601800000000027 -0.088362 rpy=-3.141590341443774 -1.515872652806505 -0.2074073356601009
- joint r_lower_leg_skin_37_fixed_joint: origin xyz=0.055257199999999985 0.0009643999999999764 -0.078318 rpy=-3.1415818045233417 -1.5231833689799856 0.007524505830633038 -> xyz=0.055257199999999985 0.0009643999999999764 -0.078318 rpy=-3.141581804523346 -1.5231833689799856 0.007524505830637575
- joint r_lower_leg_skin_46_fixed_joint: origin xyz=0.05581569999999999 0.01721639999999998 -0.05018 rpy=-3.141589878093782 -1.4275988160283246 0.3256077108756132 -> xyz=0.05581569999999999 0.01721639999999998 -0.05018 rpy=-3.141589878093782 -1.427598816028325 0.3256077108756139
- joint r_lower_leg_skin_49_fixed_joint: origin xyz=0.04113139 0.03243849999999996 -0.138859 rpy=-3.141589347506919 -1.489961356950246 0.729763592113092 -> xyz=0.04113139 0.03243849999999996 -0.138859 rpy=-3.1415893475069114 -1.4899613569502463 0.7297635921130861
- joint r_lower_leg_skin_4_fixed_joint: origin xyz=0.05831029999999999 0.016783599999999996 0.007272000000000001 rpy=-2.9863636151870843e-07 -1.256367488755018 -2.758923800870981 -> xyz=0.05831029999999999 0.016783599999999996 0.007272000000000001 rpy=-2.986363608007526e-07 -1.256367488755018 -2.7589238008709818
- joint r_lower_leg_skin_52_fixed_joint: origin xyz=0.052998339999999984 0.001266399999999973 -0.11689500000000003 rpy=-3.1415916404202857 -1.5031867442105085 0.010871726099418466 -> xyz=0.052998339999999984 0.001266399999999973 -0.11689500000000003 rpy=-3.141591640420276 -1.5031867442105085 0.010871726099408735
- joint r_lower_leg_skin_55_fixed_joint: origin xyz=0.04350267899999998 -0.030488900000000027 -0.13814300000000007 rpy=3.1415890648626297 -1.4899578703820784 -0.5972199437885269 -> xyz=0.04350267899999998 -0.030488900000000027 -0.13814300000000007 rpy=3.1415890648626297 -1.4899578703820782 -0.5972199437885254
- joint r_lower_leg_skin_6_fixed_joint: origin xyz=0.05208553999999999 0.03044339999999999 -0.022148999999999974 rpy=-3.1415892795257605 -1.4678512341064953 0.8374928890768593 -> xyz=0.05208553999999999 0.03044339999999999 -0.022148999999999974 rpy=-3.1415892795257623 -1.4678512341064949 0.8374928890768587

Commit message: Automatic build of iRonCub_Model.urdf - Triggered by a2c1cea

File: models/iRonCub-Mk1_1_v1/iRonCub/robots/iRonCub-Mk1_1_Gazebo_v1/model_stl.urdf (robot description, URDF)
Before this commit: robot iCub, 97 links, 96 joints
Joints:
- joint imu_frame_fixed_joint: origin xyz=0.009500000190735 0.13344313685842288 0.00929998892871537 rpy=3.141592653589793 1.5707962897917267 -1.5707963267948966 -> xyz=0.009500000190735 0.13344313685842288 0.00929998892871537 rpy=3.141592653589793 1.570796289791727 -1.5707963237945508
- joint l_arm_ft_sensor: origin xyz=0.05093014324520241 0 0.029175829465898032 rpy=0 -1.3089969894682862 3.1415926535896137 -> xyz=0.05093014324520241 0 0.029175829465898032 rpy=0 -1.3089969894682865 3.1415926535896164
- joint l_elbow: origin xyz=0 -0.020000000368329995 0.07925999990705779 rpy=0 -1.308996989468288 -3.1415926535896834 -> xyz=0 -0.02000000036832994 0.0792599999070578 rpy=0 -1.3089969894682885 -3.1415926535896865
- joint l_hip_roll: origin xyz=0 0.04409999999999999 0 rpy=0 0 0 -> xyz=0 0.044099999999999986 0 rpy=0 0 0
- joint l_leg_ft_sensor: origin xyz=-0.0008301999999999962 7.519999999998361e-05 -0.07429999999999995 rpy=3.141592653589793 0 0 -> xyz=-0.0008301999999999962 7.519999999999749e-05 -0.07429999999999995 rpy=3.141592653589793 0 0
- joint l_shoulder_roll: axis -0.2588190174889569 -1.0645723802156837e-17 0.9659259953138496 -> -0.2588190174889569 -1.1253323287226445e-17 0.9659259953138497
- joint l_shoulder_yaw: axis 0.9659258393523219 -5.743038501910067e-15 0.2588189963497913 -> 0.9659258393523219 -5.74303850210394e-15 0.2588189963497913; origin xyz=0.025313329844247154 1.2922216939548203e-07 -0.005396821114290115 rpy=-0.2526895449300091 -0.00851861944331826 -0.06703989350788468 -> xyz=0.025313329844247154 1.2922216940935982e-07 -0.005396821114290115 rpy=-0.2526895449300091 -0.00851861944331826 -0.06703989350788468
- joint neck_roll: axis 0.0 1.8017532951719595e-10 0.9999999628183934 -> 0.0 1.8017533007091882e-10 0.9999999628183933
- joint neck_yaw: axis 0.0 0.9999999628183934 -1.8017532951719595e-10 -> 0.0 0.9999999628183934 -1.8017532951839303e-10
- joint r_elbow_turbine: origin xyz=-0.25731143930868927 0.07362600000000005 0.09741646806310904 rpy=1.291296957309416 -0.3534717274196087 -1.4717699551817651 -> xyz=-0.25731143930868927 0.07362600000000007 0.09741646806310904 rpy=1.291296957309416 -0.3534717274196087 -1.4717699551817651
- joint r_jet_turbine: origin xyz=-0.169999999809265 -0.1141002 -0.1158885 rpy=-1.5707963207923927 -0.9424794397774842 -3.141592651408038 -> xyz=-0.169999999809265 -0.1141002 -0.1158885 rpy=-1.5707963207923916 -0.9424794397774846 -3.1415926514080383
- joint r_lower_leg_skin_14_fixed_joint: origin xyz=0.05504769999999998 -0.031175900000000006 -0.02190000000000003 rpy=-3.1415918188482506 -1.46502735635212 -0.6540334071673009 -> xyz=0.05504769999999998 -0.031175900000000006 -0.02190000000000003 rpy=-3.141591818848249 -1.4650273563521197 -0.6540334071673023
- joint r_lower_leg_skin_17_fixed_joint: origin xyz=0.027874999999999976 -0.05031190000000001 -0.023882000000000014 rpy=-3.1415645262018144 -1.5636624023748111 -1.180225087558763 -> xyz=0.027874999999999976 -0.05031190000000001 -0.023882000000000014 rpy=-3.141564526201752 -1.563662402374811 -1.1802250875588731
- joint r_lower_leg_skin_19_fixed_joint: origin xyz=0.03575341 0.041062799999999997 0.006064999999999987 rpy=-8.908777145556939e-07 -1.434986969778283 -2.158636180167247 -> xyz=0.03575341 0.041062799999999997 0.006064999999999987 rpy=-8.908777174257102e-07 -1.4349869697782824 -2.1586361801672447
- joint r_lower_leg_skin_20_fixed_joint: origin xyz=0.0234419 0.047990799999999986 -0.004952000000000012 rpy=-3.2055655052862463e-06 -1.500155130307231 -1.867550924125001 -> xyz=0.0234419 0.047990799999999986 -0.004952000000000012 rpy=-3.2055654966350685e-06 -1.5001551303072314 -1.8675509241250097
- joint r_lower_leg_skin_21_fixed_joint: origin xyz=0.024270400000000004 0.04853779999999998 -0.024276999999999993 rpy=2.2967114934038522e-05 -1.5554551388057167 -1.8741197231626947 -> xyz=0.024270400000000004 0.04853779999999998 -0.024276999999999993 rpy=2.2967114955750172e-05 -1.5554551388057172 -1.8741197231626954
- joint r_lower_leg_skin_31_fixed_joint: origin xyz=0.03914639999999998 -0.042270899999999986 0.006327000000000027 rpy=-6.583817537316898e-07 -1.4186494462021593 2.2085303298593018 -> xyz=0.03914639999999998 -0.042270899999999986 0.006327000000000027 rpy=-6.583817471389409e-07 -1.4186494462021593 2.2085303298592955
- joint r_lower_leg_skin_32_fixed_joint: origin xyz=0.045983029999999994 0.03258469999999997 -0.080733 rpy=-3.1415901498788155 -1.5223828979770997 0.6459403808870626 -> xyz=0.045983029999999994 0.03258469999999997 -0.080733 rpy=-3.141590149878832 -1.5223828979770995 0.6459403808870791
- joint r_lower_leg_skin_36_fixed_joint: origin xyz=0.05322409999999998 -0.015601800000000027 -0.088362 rpy=-3.141590341443774 -1.515872652806505 -0.2074073356601009 -> xyz=0.05322409999999998 -0.015601800000000027 -0.088362 rpy=-3.141590341443774 -1.5158726528065043 -0.20740733566009956
- joint r_lower_leg_skin_37_fixed_joint: origin xyz=0.055257199999999985 0.0009643999999999764 -0.078318 rpy=-3.141581804523346 -1.5231833689799856 0.007524505830637575 -> xyz=0.055257199999999985 0.0009643999999999764 -0.078318 rpy=-3.1415818045233417 -1.5231833689799856 0.007524505830633038
- joint r_lower_leg_skin_46_fixed_joint: origin xyz=0.05581569999999999 0.01721639999999998 -0.05018 rpy=-3.141589878093782 -1.427598816028325 0.3256077108756139 -> xyz=0.05581569999999999 0.01721639999999998 -0.05018 rpy=-3.141589878093782 -1.4275988160283246 0.3256077108756132
- joint r_lower_leg_skin_49_fixed_joint: origin xyz=0.04113139 0.03243849999999996 -0.138859 rpy=-3.1415893475069114 -1.4899613569502463 0.7297635921130861 -> xyz=0.04113139 0.03243849999999996 -0.138859 rpy=-3.141589347506919 -1.489961356950246 0.729763592113092
- joint r_lower_leg_skin_4_fixed_joint: origin xyz=0.05831029999999999 0.016783599999999996 0.007272000000000001 rpy=-2.986363608007526e-07 -1.256367488755018 -2.7589238008709818 -> xyz=0.05831029999999999 0.016783599999999996 0.007272000000000001 rpy=-2.9863636151870843e-07 -1.256367488755018 -2.758923800870981
- joint r_lower_leg_skin_52_fixed_joint: origin xyz=0.052998339999999984 0.001266399999999973 -0.11689500000000003 rpy=-3.141591640420276 -1.5031867442105085 0.010871726099408735 -> xyz=0.052998339999999984 0.001266399999999973 -0.11689500000000003 rpy=-3.1415916404202857 -1.5031867442105085 0.010871726099418466
- joint r_lower_leg_skin_55_fixed_joint: origin xyz=0.04350267899999998 -0.030488900000000027 -0.13814300000000007 rpy=3.1415890648626297 -1.4899578703820782 -0.5972199437885254 -> xyz=0.04350267899999998 -0.030488900000000027 -0.13814300000000007 rpy=3.1415890648626297 -1.4899578703820784 -0.5972199437885269
- joint r_lower_leg_skin_6_fixed_joint: origin xyz=0.05208553999999999 0.03044339999999999 -0.022148999999999974 rpy=-3.1415892795257623 -1.4678512341064949 0.8374928890768587 -> xyz=0.05208553999999999 0.03044339999999999 -0.022148999999999974 rpy=-3.1415892795257605 -1.4678512341064953 0.8374928890768593
